File: kicad/m2-io-emulator-board.kicad_pcb (KiCad board)
At the start: 2 copper layers, 180 x 190 mm, 119 parts, among them J1 N2550-6002-RB, J10 61300811121, J11 61301011121, J12 Pin Header 02x18 2.54mm Verti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, J13 VGA femelle, J14 VIDEO, J2 N2526-6002-RB, J3 B10P-SHF-1AA, J4 B12P-SHF-1AA, J5 B12P-SHF-1AA, J6 61300811121, J7 61300811121, J8 61300811121, J9 61300811121, SW1 TEST, SW2 SERVICE, U2 74HCT86, U3 OPA3355EA

Commit message: French translation (README, BOM, 3D models); silkscreen URL now points to this repository
Only F_Silkscreen changed in the Gerbers (checked file by file, dates ignored).

Co-Authored-By: Claude Opus 5.5 <noreply@anthropic.com>
Other:
- board text added: "Design: Nicolas Mailloux, 2026 nicolas.mailloux@micronick.com https://github.com/Maillouski/M2-IO-Emulator-Board"
- board text removed: "Design: Nicolas Mailloux, 2026 nicolas.mailloux@micronick.com https://github.com/Maillouski/Arcade-M3"
Changed lines of the file:
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@@
 		)
 	)
-	(gr_text "Design: Nicolas Mailloux, 2026 nicolas.mailloux@micronick.com\nhttps://github.com/Maillouski/Arcade-M3"
+	(gr_text "Design: Nicolas Mailloux, 2026 nicolas.mailloux@micronick.com\nhttps://github.com/Maillouski/M2-IO-Emulator-Board"
 		(at 112 161.5 0)
 		(layer "F.SilkS")
