File: kicad/m2-io-emulator-board.kicad_pcb (KiCad board)
At the start: 2 copper layers, 180 x 190 mm, 163 parts, among them J1 N2550-6002-RB, J10 61300811121, J11 61301011121, J12 Pin Header 02x18 2.54mm Verti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, J13 VGA femelle, J14 VIDEO, J15 HDMI A, J16 RCJ-2223, J2 N2526-6002-RB, J3 B10P-SHF-1AA, J4 B12P-SHF-1AA, J5 B12P-SHF-1AA, J6 61300811121, J7 61300811121, J8 61300811121, J9 61300811121, SW1 TEST, SW2 SERVICE, U1 ULN2803A, U2 74HCT86, U3 OPA3355EA, U4 CS5213, U5 NX3303X, U6 AT24C02, U7 TS5V330, U8 74HCT157

Commit message: Silkscreen credits: Tomi Engdahl (composite sync) and Zebidee (ArcadeControls.com forum); README credits (EN/FR); 3D model of the RCA jack J16 now 12 mm deep (body + rear cover, per datasheet), no stray pin; Gerbers, zip and renders updated
Co-Authored-By: Claude Opus 5.5 <noreply@anthropic.com>
Other:
- board text added: "ArcadeControls.com forum: Zebidee"
- board text added: "Composite sync: Tomi Engdahl"
Changed lines of the file:
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@@
 		)
 	)
+	(gr_text "Composite sync: Tomi Engdahl"
+		(at 104.5 160.4 0)
+		(layer "F.SilkS")
+		(effects
+			(font
+				(size 1.3 1.3)
+				(thickness 0.169)
+			)
+			(justify left bottom)
+		)
+	)
+	(gr_text "ArcadeControls.com forum: Zebidee"
+		(at 104.5 162.48 0)
+		(layer "F.SilkS")
+		(effects
+			(font
+				(size 1.3 1.3)
+				(thickness 0.169)
+			)
+			(justify left bottom)
+		)
+	)
 	(gr_text "Thanks to all. Not affiliated with or endorsed by SEGA."
-		(at 104.5 162 0)
+		(at 104.5 166.16 0)
 		(layer "F.SilkS")
 		(effects
@@
 	)
 	(group "Credits"
-		(members "32a9a2c8-ebb0-402e-b8e9-d7f498fcf1ff" "3cad0f6f-129b-4547-84f6-fd7b006853b1"
-			"44f3a08a-5582-4395-a4df-08e05cad2e52" "6ac56ea5-e75b-4cf4-aa95-8f2c93eaff0a"
+		(members "28d9f870-f887-473d-9ab6-00d0c723b274" "32a9a2c8-ebb0-402e-b8e9-d7f498fcf1ff"
+			"3cad0f6f-129b-4547-84f6-fd7b006853b1" "44f3a08a-5582-4395-a4df-08e05cad2e52"
+			"4880c8bd-ffef-4bb3-b9bd-a2d4894de5c7" "6ac56ea5-e75b-4cf4-aa95-8f2c93eaff0a"
 			"833a4af0-08af-4443-a8b4-0bb6a1fe6a5d" "9e0b8de9-4437-40ec-ac01-3bc5f5d61a7f"
 			"a81e32e6-4828-4e4f-b450-9f6c2e7c89ea" "b1936d7d-1726-4446-ab91-e27d5365dd63"
 			"b6d0365f-5223-4756-8d10-bb64816138ab" "d386013a-1502-47ac-869a-e45ab31ca66e"
-			"f89d1cb5-9a34-41b8-b62e-c91d0bb3d21e"
+			"e17899e1-3fa9-4c21-9742-f97e0d4d9e09" "f89d1cb5-9a34-41b8-b62e-c91d0bb3d21e"
 		)
 	)
