File: kicad/m2-io-emulator-board.kicad_pcb (KiCad board)
At the start: 2 copper layers, 180 x 190 mm, 163 parts, among them J1 N2550-6002-RB, J10 61300811121, J11 61301011121, J12 Pin Header 02x18 2.54mm Verti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, J13 VGA femelle, J14 VIDEO, J15 HDMI A, J16 RCJ-2223, J2 N2526-6002-RB, J3 B10P-SHF-1AA, J4 B12P-SHF-1AA, J5 B12P-SHF-1AA, J6 61300811121, J7 61300811121, J8 61300811121, J9 61300811121, SW1 TEST, SW2 SERVICE, U1 ULN2803A, U2 74HCT86, U3 OPA3355EA, U4 CS5213, U5 NX3303X, U6 AT24C02, U7 TS5V330, U8 74HCT157

Commit message: V3.2: J16 footprint fits the Same Sky RCJ-2223 or the Lian Xin XDJK-0271-1650 (LCSC C7527522, in stock at JLCPCB); top jack = left, bottom = right; J16 moved 2.25 mm; U4 exposed-pad vias filled and capped in the design; silkscreen V3.2; Gerbers, zip, position file, schematic PDF and 3D renders regenerated
Parts:
- J16: value RCJ-2223 -> XDJK-0271-1650; footprint interface-borne:CUI_RCJ-22xx_RCA_Dual_Horizontal -> interface-borne:RCA_Dual_Stacked_RCJ-22xx_XDJK-0271-1650
- moved J16 2.25 mm to (8.20, 177.8)
Connections:
- J16 pad 2: /AUD_OUT_L -> /AUD_OUT_R
- J16 pad 3: /AUD_OUT_R -> /AUD_OUT_L
Routing:
- net /AUD_OUT_L: track 4.25 -> 12.2 mm, vias 0 -> 1
- net /AUD_OUT_R: track 3.00 -> 7.40 mm
- net /GND: track 336.5 -> 339.6 mm
- net /CS_3V3: track 24.9 -> 26.0 mm
- net /HD_B: track 67.2 -> 68.1 mm
Other:
- board text added: "V3.2"
- board text removed: "V3"
