File: kicad/m2-io-emulator-board.kicad_sch (KiCad schematic)
At the start: 163 parts, among them J1 N2550-6002-RB, J10 61300811121, J11 61301011121, J12 Pin Header 02x18 2.54mm Verti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, J13 VGA femelle, J14 VIDEO, J15 HDMI A, J16 RCJ-2223, J2 N2526-6002-RB, J3 B10P-SHF-1AA, J4 B12P-SHF-1AA, J5 B12P-SHF-1AA, J6 61300811121, J7 61300811121, J8 61300811121, J9 61300811121, SW1 TEST, SW2 SERVICE, U1 ULN2803A, U2 74HCT86, U3 OPA3355EA, U4 CS5213, U5 NX3303X, U6 AT24C02, U7 TS5V330, U8 74HCT157

Commit message: V3: polarity-independent composite sync (Tomi Engdahl's circuit: R66/R67 + C47/C48, all 4 gates of U2), EDID EEPROM U6 and C24 now fitted, "V3" and "24kHz" on the silkscreen; Gerbers, drill files, schematic PDF, 3D renders, BOM (EN/FR) and JLCPCB files (121 SMD) updated
Parts:
- added C47, C48: 22 µF, Capacitor_SMD:C_0805_2012Metric, symbol Device:C
- added R66, R67: 2,2 kΩ, Resistor_SMD:R_0805_2012Metric, symbol Device:R
- C24, U6: now fitted
Connections:
- net +5V_MEGA: now also U2.10 (3B); no longer U2.5 (2B)
- net CSYNC_N: now also U2.8 (3Y); no longer U2.6 (2Y)
- net CSYNC_XOR: now also U2.11 (4Y), U2.9 (3A); no longer U2.3 (1Y), U2.4 (2A)
- net GND: now also C47.2, C48.2; no longer U2.10 (3B), U2.12 (4A), U2.13 (4B), U2.9 (3A)
- net VGA_HS: now also R66.1
- net VGA_VS: now also U2.5 (2B), R67.1; no longer U2.2 (1B)
- new net HS_AVG: C47.1, R66.2, U2.2 (1B)
- new net HS_NORM: U2.13 (4B), U2.3 (1Y)
- new net VS_AVG: C48.1, R67.2, U2.4 (2A)
- new net VS_NORM: U2.12 (4A), U2.6 (2Y)
- no-connect marks 129 -> 127
Other:
- note added: "V3 (2026-10-16) : synchro indépendante de la polarité (T. Engdahl). U2 portes 1-2 : chaque synchro XOR sa moyenne (2,2 kΩ / 22 µF) → HS_NORM, VS_NORM en impulsions positives → porte 4 → porte 3 (inversion) : CSYNC négative quelles que soient les polarités H/V."
Changed lines of the file:
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@@
 	)
 	(no_connect
-		(at 114.3 533.4)
-	)
-	(no_connect
 		(at 167.64 680.72)
 	)
@@
 	)
 	(no_connect
-		(at 114.3 525.78)
-	)
-	(no_connect
 		(at 88.9 187.96)
 	)
@@
 		)
 	)
-	(label "VGA_VS"
+	(label "HS_AVG"
 		(at 114.3 510.54 180)
 		(effects
@@
 		)
 	)
-	(label "CSYNC_XOR"
+	(label "VS_AVG"
 		(at 114.3 515.62 180)
 		(effects
@@
 		)
 	)
-	(label "GND"
+	(label "VS_NORM"
 		(at 114.3 535.94 180)
 		(effects
@@
 		)
 	)
-	(label "GND"
+	(label "HS_NORM"
 		(at 114.3 538.48 180)
 		(effects
@@
 		)
 	)
-	(label "CSYNC_XOR"
+	(label "HS_NORM"
 		(at 114.3 513.08 180)
 		(effects
@@
 		)
 	)
-	(label "+5V_MEGA"
+	(label "VGA_VS"
 		(at 114.3 518.16 180)
 		(effects
@@
 		)
 	)
-	(label "GND"
+	(label "CSYNC_XOR"
 		(at 114.3 528.32 180)
 		(effects
@@
 		)
 	)
-	(label "CSYNC_N"
+	(label "VS_NORM"
 		(at 114.3 520.7 180)
 		(effects
@@
 		)
 	)
-	(label "GND"
+	(label "+5V_MEGA"
 		(at 114.3 530.86 180)
 		(effects
@@
 		(on_board yes)
 		(in_pos_files yes)
-		(dnp yes)
+		(dnp no)
 		(property "Reference" "C24"
 			(at 741.68 621.03 0)
@@
 		(on_board yes)
 		(in_pos_files yes)
-		(dnp yes)
+		(dnp no)
 		(property "Reference" "U6"
 			(at 886.46 429.26 0)
@@
 		)
 	)
+	(label "CSYNC_N" (at 114.3 525.78 180) (effects (font (size 1.27 1.27)) (justify right bottom)))
+	(label "CSYNC_XOR" (at 114.3 533.4 180) (effects (font (size 1.27 1.27)) (justify right bottom)))
+	(text "V3 (2026-10-16) : synchro indépendante de la polarité (T. Engdahl).\nU2 portes 1-2 : chaque synchro XOR sa moyenne (2,2 kΩ / 22 µF)\n→ HS_NORM, VS_NORM en impulsions positives → porte 4 → porte 3 (inversion) :\nCSYNC négative quelles que soient les polarités H/V." (exclude_from_sim no) (at 72.39 560.07 0) (effects (font (size 1.27 1.27)) (justify left bottom)))
+(symbol (lib_id "Device:R") (at 73.66 508.00 0) (unit 1) (body_style 1) (exclude_from_sim no) (in_bom yes) (on_board yes) (dnp no)
+(property "Reference" "R66" (at 76.20 506.73 0) (effects (font (size 1.27 1.27)) (justify left)))
+(property "Value" "2,2 kΩ" (at 76.20 509.27 0) (effects (font (size 1.27 1.27)) (justify left)))
+(property "Footprint" "Resistor_SMD:R_0805_2012Metric" (at 73.66 508.00 0) (effects (font (size 1.27 1.27))) (hide yes))
+(property "Datasheet" "" (at 73.66 508.00 0) (effects (font (size 1.27 1.27))) (hide yes))
+(property "MPN" "RC0805FR-072K2L" (at 73.66 508.00 0) (effects (font (size 1.27 1.27))) (hide yes))
+(pin "1")(pin "2")
+(instances (project "m2-io-emulator-board" (path "/d44661bf-d01e-4075-8845-9c2310b0d4a5" (reference "R66") (unit 1)))))
+(label "VGA_HS" (at 73.66 504.19 90) (effects (font (size 1.27 1.27)) (justify left bottom)))
+(label "HS_AVG" (at 73.66 511.81 270) (effects (font (size 1.27 1.27)) (justify right bottom)))
+(symbol (lib_id "Device:C") (at 91.44 508.00 0) (unit 1) (body_style 1) (exclude_from_sim no) (in_bom yes) (on_board yes) (dnp no)
+(property "Reference" "C47" (at 93.98 506.73 0) (effects (font (size 1.27 1.27)) (justify left)))
+(property "Value" "22 µF" (at 93.98 509.27 0) (effects (font (size 1.27 1.27)) (justify left)))
+(property "Footprint" "Capacitor_SMD:C_0805_2012Metric" (at 91.44 508.00 0) (effects (font (size 1.27 1.27))) (hide yes))
+(property "Datasheet" "" (at 91.44 508.00 0) (effects (font (size 1.27 1.27))) (hide yes))
+(property "MPN" "GRM21BR61E226ME44L" (at 91.44 508.00 0) (effects (font (size 1.27 1.27))) (hide yes))
+(pin "1")(pin "2")
+(instances (project "m2-io-emulator-board" (path "/d44661bf-d01e-4075-8845-9c2310b0d4a5" (reference "C47") (unit 1)))))
+(label "HS_AVG" (at 91.44 504.19 90) (effects (font (size 1.27 1.27)) (justify left bottom)))
+(label "GND" (at 91.44 511.81 270) (effects (font (size 1.27 1.27)) (justify right bottom)))
+(symbol (lib_id "Device:R") (at 73.66 535.94 0) (unit 1) (body_style 1) (exclude_from_sim no) (in_bom yes) (on_board yes) (dnp no)
+(property "Reference" "R67" (at 76.20 534.67 0) (effects (font (size 1.27 1.27)) (justify left)))
+(property "Value" "2,2 kΩ" (at 76.20 537.21 0) (effects (font (size 1.27 1.27)) (justify left)))
+(property "Footprint" "Resistor_SMD:R_0805_2012Metric" (at 73.66 535.94 0) (effects (font (size 1.27 1.27))) (hide yes))
+(property "Datasheet" "" (at 73.66 535.94 0) (effects (font (size 1.27 1.27))) (hide yes))
+(property "MPN" "RC0805FR-072K2L" (at 73.66 535.94 0) (effects (font (size 1.27 1.27))) (hide yes))
+(pin "1")(pin "2")
+(instances (project "m2-io-emulator-board" (path "/d44661bf-d01e-4075-8845-9c2310b0d4a5" (reference "R67") (unit 1)))))
+(label "VGA_VS" (at 73.66 532.13 90) (effects (font (size 1.27 1.27)) (justify left bottom)))
+(label "VS_AVG" (at 73.66 539.75 270) (effects (font (size 1.27 1.27)) (justify right bottom)))
+(symbol (lib_id "Device:C") (at 91.44 535.94 0) (unit 1) (body_style 1) (exclude_from_sim no) (in_bom yes) (on_board yes) (dnp no)
+(property "Reference" "C48" (at 93.98 534.67 0) (effects (font (size 1.27 1.27)) (justify left)))
+(property "Value" "22 µF" (at 93.98 537.21 0) (effects (font (size 1.27 1.27)) (justify left)))
+(property "Footprint" "Capacitor_SMD:C_0805_2012Metric" (at 91.44 535.94 0) (effects (font (size 1.27 1.27))) (hide yes))
+(property "Datasheet" "" (at 91.44 535.94 0) (effects (font (size 1.27 1.27))) (hide yes))
+(property "MPN" "GRM21BR61E226ME44L" (at 91.44 535.94 0) (effects (font (size 1.27 1.27))) (hide yes))
+(pin "1")(pin "2")
+(instances (project "m2-io-emulator-board" (path "/d44661bf-d01e-4075-8845-9c2310b0d4a5" (reference "C48") (unit 1)))))
+(label "VS_AVG" (at 91.44 532.13 90) (effects (font (size 1.27 1.27)) (justify left bottom)))
+(label "GND" (at 91.44 539.75 270) (effects (font (size 1.27 1.27)) (justify right bottom)))
 	(sheet_instances
 		(path "/"
