File: kicad/m2-io-emulator-board.kicad_sch (KiCad schematic)
At the start: 167 parts, among them J1 N2550-6002-RB, J10 61300811121, J11 61301011121, J12 Pin Header 02x18 2.54mm Verti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, J13 VGA femelle, J14 VIDEO, J15 HDMI A, J16 RCJ-2223, J2 N2526-6002-RB, J3 B10P-SHF-1AA, J4 B12P-SHF-1AA, J5 B12P-SHF-1AA, J6 61300811121, J7 61300811121, J8 61300811121, J9 61300811121, SW1 TEST, SW2 SERVICE, U1 ULN2803A, U2 74HCT86, U3 OPA3355EA, U4 CS5213, U5 NX3303X, U6 AT24C02, U7 TS5V330, U8 74HCT157

Commit message: BOM: in-stock replacements for the 10 µF and 22 µF capacitors, C17, R47 and J15 (DigiKey, checked 2026-10-16); JST NH headers from LCSC; schematic MPN fields updated
Co-Authored-By: Claude Opus 5.5 <noreply@anthropic.com>
Parts:
- C17: MPN EEU-FC1C101 -> EEU-FC1C101H
- C19, C23, C25, C26, C30, C32, C34, C37, C41, C42, C45: MPN CL21B106KOQNNNG -> CL21A106KAYNNNE
- C47, C48: MPN GRM21BR61E226ME44L -> CL21A226MOCLRNC
- R47: MPN RC0805FR-07470RL -> RMCF0805FT470R
Changed lines of the file:
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@@
 			)
 		)
-		(property "MPN" "CL21B106KOQNNNG"
+		(property "MPN" "CL21A106KAYNNNE"
 			(at 767.08 688.34 0)
 			(hide yes)
@@
 			)
 		)
-		(property "MPN" "RC0805FR-07470RL"
+		(property "MPN" "RMCF0805FT470R"
 			(at 256.54 518.16 0)
 			(hide yes)
@@
 			)
 		)
-		(property "MPN" "EEU-FC1C101"
+		(property "MPN" "EEU-FC1C101H"
 			(at 477.52 88.9 0)
 			(hide yes)
@@
 			)
 		)
-		(property "MPN" "CL21B106KOQNNNG"
+		(property "MPN" "CL21A106KAYNNNE"
 			(at 739.14 655.32 0)
 			(hide yes)
@@
 			)
 		)
-		(property "MPN" "CL21B106KOQNNNG"
+		(property "MPN" "CL21A106KAYNNNE"
 			(at 767.08 622.3 0)
 			(hide yes)
@@
 			)
 		)
-		(property "MPN" "CL21B106KOQNNNG"
+		(property "MPN" "CL21A106KAYNNNE"
 			(at 795.02 622.3 0)
 			(hide yes)
@@
 			)
 		)
-		(property "MPN" "CL21B106KOQNNNG"
+		(property "MPN" "CL21A106KAYNNNE"
 			(at 906.78 622.3 0)
 			(hide yes)
@@
 			)
 		)
-		(property "MPN" "CL21B106KOQNNNG"
+		(property "MPN" "CL21A106KAYNNNE"
 			(at 795.02 655.32 0)
 			(hide yes)
@@
 			)
 		)
-		(property "MPN" "CL21B106KOQNNNG"
+		(property "MPN" "CL21A106KAYNNNE"
 			(at 878.84 655.32 0)
 			(hide yes)
@@
 			)
 		)
-		(property "MPN" "CL21B106KOQNNNG"
+		(property "MPN" "CL21A106KAYNNNE"
 			(at 533.4 88.9 0)
 			(hide yes)
@@
 			)
 		)
-		(property "MPN" "CL21B106KOQNNNG"
+		(property "MPN" "CL21A106KAYNNNE"
 			(at 878.84 688.34 0)
 			(hide yes)
@@
 			)
 		)
-		(property "MPN" "CL21B106KOQNNNG"
+		(property "MPN" "CL21A106KAYNNNE"
 			(at 795.02 688.34 0)
 			(hide yes)
@@
 			)
 		)
-		(property "MPN" "CL21B106KOQNNNG"
+		(property "MPN" "CL21A106KAYNNNE"
 			(at 162.56 749.3 0)
 			(hide yes)
@@
 (property "Footprint" "Capacitor_SMD:C_0805_2012Metric" (at 91.44 508.00 0) (effects (font (size 1.27 1.27))) (hide yes))
 (property "Datasheet" "" (at 91.44 508.00 0) (effects (font (size 1.27 1.27))) (hide yes))
-(property "MPN" "GRM21BR61E226ME44L" (at 91.44 508.00 0) (effects (font (size 1.27 1.27))) (hide yes))
+(property "MPN" "CL21A226MOCLRNC" (at 91.44 508.00 0) (effects (font (size 1.27 1.27))) (hide yes))
 (pin "1")(pin "2")
 (instances (project "m2-io-emulator-board" (path "/d44661bf-d01e-4075-8845-9c2310b0d4a5" (reference "C47") (unit 1)))))
@@
 (property "Footprint" "Capacitor_SMD:C_0805_2012Metric" (at 91.44 535.94 0) (effects (font (size 1.27 1.27))) (hide yes))
 (property "Datasheet" "" (at 91.44 535.94 0) (effects (font (size 1.27 1.27))) (hide yes))
-(property "MPN" "GRM21BR61E226ME44L" (at 91.44 535.94 0) (effects (font (size 1.27 1.27))) (hide yes))
+(property "MPN" "CL21A226MOCLRNC" (at 91.44 535.94 0) (effects (font (size 1.27 1.27))) (hide yes))
 (pin "1")(pin "2")
 (instances (project "m2-io-emulator-board" (path "/d44661bf-d01e-4075-8845-9c2310b0d4a5" (reference "C48") (unit 1)))))
