File: kicad/m2-io-emulator-board.kicad_sch (KiCad schematic)
At the start: 167 parts, among them J1 N2550-6002-RB, J10 61300811121, J11 61301011121, J12 Pin Header 02x18 2.54mm Verti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, J13 VGA femelle, J14 VIDEO, J15 HDMI A, J16 RCJ-2223, J2 N2526-6002-RB, J3 B10P-SHF-1AA, J4 B12P-SHF-1AA, J5 B12P-SHF-1AA, J6 61300811121, J7 61300811121, J8 61300811121, J9 61300811121, SW1 TEST, SW2 SERVICE, U1 ULN2803A, U2 74HCT86, U3 OPA3355EA, U4 CS5213, U5 NX3303X, U6 AT24C02, U7 TS5V330, U8 74HCT157

Commit message: V3.2: J16 footprint fits the Same Sky RCJ-2223 or the Lian Xin XDJK-0271-1650 (LCSC C7527522, in stock at JLCPCB); top jack = left, bottom = right; J16 moved 2.25 mm; U4 exposed-pad vias filled and capped in the design; silkscreen V3.2; Gerbers, zip, position file, schematic PDF and 3D renders regenerated
Parts:
- J16: value RCJ-2223 -> XDJK-0271-1650; footprint interface-borne:CUI_RCJ-22xx_RCA_Dual_Horizontal -> interface-borne:RCA_Dual_Stacked_RCJ-22xx_XDJK-0271-1650; MPN RCJ-2223 -> XDJK-0271-1650
Connections:
- net AUD_OUT_L: now also J16.3 (X1_HAUT); no longer J16.2 (X2_BAS)
- net AUD_OUT_R: now also J16.2 (X2_BAS); no longer J16.3 (X1_HAUT)
Changed lines of the file:
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@@
 		)
 	)
-	(label "AUD_OUT_R"
+	(label "AUD_OUT_L"
 		(at 822.96 546.1 180)
 		(effects
@@
 		)
 	)
-	(label "AUD_OUT_L"
+	(label "AUD_OUT_R"
 		(at 822.96 543.56 180)
 		(effects
@@
 			)
 		)
-		(property "Value" "RCJ-2223"
+		(property "Value" "XDJK-0271-1650"
 			(at 828.04 551.18 0)
 			(show_name no)
@@
 			)
 		)
-		(property "Footprint" "interface-borne:CUI_RCJ-22xx_RCA_Dual_Horizontal"
+		(property "Footprint" "interface-borne:RCA_Dual_Stacked_RCJ-22xx_XDJK-0271-1650"
 			(at 828.04 538.48 0)
 			(hide yes)
@@
 			)
 		)
-		(property "Description" "Sortie audio de la puce HDMI vers le préampli : prise du haut rouge = DROITE, prise du bas blanche = GAUCHE"
+		(property "Description" "Sortie audio de la puce HDMI vers le préampli : prise du haut (broche 3) = GAUCHE, prise du bas (broche 2) = DROITE. XDJK-0271-1650 (JLCPCB C7527522) : haut blanc, bas rouge. RCJ-2223 (DigiKey) : haut rouge = GAUCHE"
 			(at 828.04 538.48 0)
 			(hide yes)
@@
 			)
 		)
-		(property "MPN" "RCJ-2223"
+		(property "MPN" "XDJK-0271-1650"
 			(at 828.04 538.48 0)
 			(hide yes)
